Commit message: Add imu, gnss, lidar links

File: src/misc/johnny_description/urdf/johnny.urdf.xacro (robot description, xacro)
@@ -120,9 +120,21 @@
         </visual>
     </link>
+    <link name="gnss_link" />
+    <joint name="gnss_link_joint" type="fixed">
+        <origin xyz="0 0 1.76" rpy="0 0 0" />
+        <parent link="base_link" />
+        <child link="gnss_link" />
+    </joint>
     <link name="imu_link" />
     <joint name="imu_link_joint" type="fixed">
-        <origin xyz="0 0 0" rpy="0 0 0" />
+        <origin xyz="0 0 1.76" rpy="0 0 0" />
         <parent link="base_link" />
         <child link="imu_link" />
     </joint>
+    <link name="lidar_link" />
+    <joint name="lidar_link_joint" type="fixed">
+        <origin xyz="0.37 0 1.31" rpy="0 ${PI/6} 0" />
+        <parent link="base_link" />
+        <child link="lidar_link" />
+    </joint>
 </robot>

Commit message: Add joint_state_publisher

File: src/misc/johnny_description/urdf/johnny.urdf.xacro (robot description, xacro)
@@ -2,11 +2,12 @@
 <robot name="warthog" xmlns:xacro="http://www.ros.org/wiki/xacro">
     <xacro:property name="PI" value="3.1415926535897931" />
-    <xacro:property name="wheel_radius" value="0.3" />
-    <xacro:property name="wheel_width" value="0.25" />
+    <xacro:property name="wheel_radius" value="0.216" />
+    <xacro:property name="wheel_width" value="0.114" />
     <xacro:property name="wheel_mass" value="15" />
     <xacro:property name="wheel_to_track_ratio" value="0.5962" />
-    <xacro:property name="axle_x_offset" value="0.457367" />
-    <xacro:property name="axle_y_offset" value="0.0" />
-    <xacro:property name="axle_z_offset" value="-0.012977" />
+    <xacro:property name="axle_x_offset" value="0.395" />
+    <xacro:property name="axle_y_offset" value="0.765" />
+    <!-- base_link is on the ground plane, so the wheel axle is {wheel_radius} above it. -->
+    <xacro:property name="axle_z_offset" value="${wheel_radius}" />
     <xacro:property name="diff_unit_length" value="1.34" />
     <xacro:property name="diff_unit_width" value="0.28" />
@@ -77,5 +78,5 @@
                 <xacro:wheel_inertia m="${wheel_mass}" r="${wheel_radius}" h="${wheel_width}" />
             </inertial>
-            <visual>
+            <!-- <visual>
                 <origin xyz="0 0 0" rpy="0 0 ${PI/2}" />
                 <geometry>
@@ -83,5 +84,5 @@
                 </geometry>
                 <material name="white" />
-            </visual>
+            </visual> -->
             <collision>
                 <origin xyz="0 0 0" rpy="${PI/2} 0 0" />

Commit message: Add xarm_description package, with most unneeded files removed

File: src/misc/johnny_description/urdf/johnny.urdf.xacro (robot description, xacro)
@@ -22,4 +22,6 @@
     <xacro:property name="chassis_mass" value="100" />
     <xacro:property name="dummy_inertia" value="1e-09" />
+    <!-- Include the xarm6 urdf -->
+    <xacro:include filename="$(find xarm_description)/urdf/xarm_device_macro.xacro" />
     <!--
     Optional paint colors.
@@ -139,3 +141,10 @@
         <child link="lidar_link" />
     </joint>
+    <link name="arm_link" />
+    <joint name="arm_link_joint" type="fixed">
+        <origin xyz="1.25 0 1.0" rpy="0 ${PI/2} 0" />
+        <parent link="base_link" />
+        <child link="arm_link" />
+    </joint>
+    <xacro:xarm_device dof="6" attach_to="arm_link" add_gripper="true" />
 </robot>

Commit message: Update joint_state_publisher to listen to joint state from EcoSim

File: src/misc/johnny_description/urdf/johnny.urdf.xacro (robot description, xacro)
@@ -143,5 +143,5 @@
     <link name="arm_link" />
     <joint name="arm_link_joint" type="fixed">
-        <origin xyz="1.25 0 1.0" rpy="0 ${PI/2} 0" />
+        <origin xyz="0.75 0 0.75" rpy="0 ${PI/2} 0" />
         <parent link="base_link" />
         <child link="arm_link" />

Commit message: Add collision meshes for multi eef

File: src/misc/johnny_description/urdf/johnny.urdf.xacro (robot description, xacro)
@@ -147,4 +147,24 @@
         <child link="arm_link" />
     </joint>
-    <xacro:xarm_device dof="6" attach_to="arm_link" add_gripper="true" />
+    <xacro:xarm_device dof="6" attach_to="arm_link" add_gripper="false" />
+    <link name="gripper_link">
+        <visual>
+            <origin xyz="0 0 0" rpy="0 0 0" />
+            <geometry>
+                <mesh filename="package://johnny_description/meshes/multi_eef.obj" />
+            </geometry>
+            <material name="light_grey" />
+        </visual>
+        <collision>
+            <origin xyz="0 0 0" rpy="0 0 0" />
+            <geometry>
+                <mesh filename="package://johnny_description/meshes/multi_eef_collision.obj" />
+            </geometry>
+        </collision>
+    </link>
+    <joint name="gripper_link_joint" type="fixed">
+        <origin xyz="0 0 0" rpy="0 0 0" />
+        <parent link="link_eef" />
+        <child link="gripper_link" />
+    </joint>
 </robot>

Commit message: Add gripper_link, the midpoint between the fingers

File: src/misc/johnny_description/urdf/johnny.urdf.xacro (robot description, xacro)
@@ -148,5 +148,5 @@
     </joint>
     <xacro:xarm_device dof="6" attach_to="arm_link" add_gripper="false" />
-    <link name="gripper_link">
+    <link name="multi_eef_link">
         <visual>
             <origin xyz="0 0 0" rpy="0 0 0" />
@@ -163,7 +163,14 @@
         </collision>
     </link>
-    <joint name="gripper_link_joint" type="fixed">
+    <joint name="multi_eef_joint" type="fixed">
         <origin xyz="0 0 0" rpy="0 0 0" />
         <parent link="link_eef" />
+        <child link="multi_eef_link" />
+    </joint>
+    <link name="gripper_link">
+    </link>
+    <joint name="gripper_joint" type="fixed">
+        <origin xyz="-0.139 0 0.125" rpy="0 ${-PI/3} 0" />
+        <parent link="multi_eef_link" />
         <child link="gripper_link" />
     </joint>

Commit message: Add very basic collision checking

File: src/misc/johnny_description/urdf/johnny.urdf.xacro (robot description, xacro)
@@ -143,5 +143,5 @@
     <link name="arm_link" />
     <joint name="arm_link_joint" type="fixed">
-        <origin xyz="0.75 0 0.75" rpy="0 ${PI/2} 0" />
+        <origin xyz="0.75 0 0.63" rpy="0 ${PI/2} 0" />
         <parent link="base_link" />
         <child link="arm_link" />

Commit message: Add visualization to trajectory planner

File: src/misc/johnny_description/urdf/johnny.urdf.xacro (robot description, xacro)
@@ -122,4 +122,10 @@
             <material name="white" />
         </visual>
+        <collision>
+            <origin xyz="0 0 0" rpy="0 0 0" />
+            <geometry>
+                <mesh filename="package://johnny_description/meshes/amiga_chassis_lowpoly.stl" />
+            </geometry>
+        </collision>
     </link>
     <link name="gnss_link" />

Commit message: Add prm generation with collision checking

File: src/misc/johnny_description/urdf/johnny.urdf.xacro (robot description, xacro)
@@ -149,5 +149,5 @@
     <link name="arm_link" />
     <joint name="arm_link_joint" type="fixed">
-        <origin xyz="0.75 0 0.63" rpy="0 ${PI/2} 0" />
+        <origin xyz="0.68 0 0.63" rpy="0 ${PI/2} 0" />
         <parent link="base_link" />
         <child link="arm_link" />
